File: Output.kicad_sch (KiCad schematic)
At the start: 108 parts, among them J10 DB301V-3.5-3P-GN, J11 DB301V-3.5-3P-GN, J12 DB301V-3.5-3P-GN, J13 DB301V-3.5-3P-GN, J14 DB301V-3.5-3P-GN, J15 DB301V-3.5-3P-GN, J16 DB301V-3.5-3P-GN, J17 DB301V-3.5-3P-GN, J18 DB301V-3.5-3P-GN, J19 DB301V-3.5-3P-GN, J20 DB301V-3.5-3P-GN, J21 DB301V-3.5-3P-GN, J22 DB301V-3.5-3P-GN, J23 DB301V-3.5-3P-GN, J24 DB301V-3.5-3P-GN, J25 DB301V-3.5-3P-GN, J26 DB301V-3.5-3P-GN, J27 DB301V-3.5-3P-GN, J28 DB301V-3.5-3P-GN, J29 DB301V-3.5-3P-GN, J30 DB301V-3.5-3P-GN, J31 DB301V-3.5-3P-GN, J32 DB301V-3.5-3P-GN, J33 DB301V-3.5-3P-GN, J34 DB301V-3.5-3P-GN, J35 DB301V-3.5-3P-GN, J36 DB301V-3.5-3P-GN, J37 DB301V-3.5-3P-GN, J39 DB301V-3.5-3P-GN, J7 DB301V-3.5-3P-GN, J8 DB301V-3.5-3P-GN, J9 DB301V-3.5-3P-GN, U10 SN74LVC8T245PWR, U11 SN74LVC8T245PWR, U7 SN74LVC8T245PWR, U8 SN74LVC8T245PWR

Commit message: Updates
Changed lines of the file:
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@@
 	(text "Series resistors go near the buffers, not the connection"
 		(exclude_from_sim no)
-		(at 96.266 170.688 0)
+		(at 95.758 179.07 0)
 		(effects
 			(font

Commit message: Fix ERC: register missing libraries, add PWR_FLAGs, rename zone rails
- Register project-local sym-lib-table/fp-lib-table. PixelBlit points at
  pico-pixel's live library; RPI_COMPILED/KiCad_Standard/EasyEDA/PCM_JLCPCB
  footprints vendored (via the abandoned universal-strip-controller-first
  attempt) into libs/; RPI_DB, RPI - Power, EasyEDA, PCM_JLCPCB-Diodes and
  PCM_JLCPCB-Resistors symbols extracted from the schematics' own embedded
  symbol cache into standalone .kicad_sym files, validated with
  `kicad-cli sym upgrade`.
- Fix U1's footprint: RPI_COMPILED:rpi_rp2350b doesn't exist anywhere
  (not even in the original RP2350B-MINIMAL reference) - corrected to
  rpi_rp2350b_vias, the footprint that's actually there.
- Point D10 (BZT52C15V) and R5/R20 (0603s) at KiCad's own standard
  SOD-123/0603 footprints; no vendored copy of their original
  EasyEDA/JLCPCB footprints existed anywhere to source from.
- Add PWR_FLAGs on the 8 nets ERC found undriven: +VIN_Z1-4, +12V_SYS,
  GND (top sheet), +1V1, and VREG_AVDD (U1 pin 61).
- Rename +12V_Z1-4 to +VIN_Z1-4 (zones carry 5-12V depending on what's
  plugged in, not a fixed 12V).

ERC: 1009 violations / 8 errors -> 533 violations / 0 errors.
Remaining warnings are pre-existing: fuse/diode symbols typed
Unspecified instead of Passive (pin_to_pin), intentional dual net
labels (STRINGn/GPIOn etc., except a real USB_D+/USB_D- issue still
open), schematic drawing hygiene (off-grid/dangling wire endpoints),
and symbol-cache drift now visible now that real libraries exist
(lib_symbol_mismatch - fix via Update Symbols from Library in KiCad).
Connections:
- net +12V_Z1 is gone; now on net +VIN_Z1: F11.1, F13.1, F15.1, F17.1, F19.1, F21.1, F23.1, F9.1
- net +12V_Z2 is gone; now on net +VIN_Z2: F10.1, F12.1, F14.1, F16.1, F18.1, F20.1, F22.1, F8.1
- net +VIN_Z1: now reaches F9.2, J8.1
- net +VIN_Z2: now reaches F8.2, J7.1
- net +12V_Z3 renamed +VIN_Z3
- net +12V_Z4 renamed +VIN_Z4

Commit message: Added footprints for resistors
Parts:
- C34, C35, C36, C37, C38, C39, C40, C41: Capacitance 100nF -> (none); capacitance (none) -> 100nF
Changed lines of the file:
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@@
 			)
 		)
-		(property "Capacitance" "100nF"
+		(property "capacitance" "100nF"
 			(at 267.97 30.48 0)
 			(hide yes)
@@
 			)
 		)
-		(property "Capacitance" "100nF"
+		(property "capacitance" "100nF"
 			(at 19.05 27.94 0)
 			(hide yes)
@@
 			)
 		)
-		(property "Capacitance" "100nF"
+		(property "capacitance" "100nF"
 			(at 260.35 30.48 0)
 			(hide yes)
@@
 			)
 		)
-		(property "Capacitance" "100nF"
+		(property "capacitance" "100nF"
 			(at 275.59 30.48 0)
 			(hide yes)
@@
 			)
 		)
-		(property "Capacitance" "100nF"
+		(property "capacitance" "100nF"
 			(at 252.73 30.48 0)
 			(hide yes)
@@
 			)
 		)
-		(property "Capacitance" "100nF"
+		(property "capacitance" "100nF"
 			(at 41.91 27.94 0)
 			(hide yes)
@@
 			)
 		)
-		(property "Capacitance" "100nF"
+		(property "capacitance" "100nF"
 			(at 26.67 27.94 0)
 			(hide yes)
@@
 			)
 		)
-		(property "Capacitance" "100nF"
+		(property "capacitance" "100nF"
 			(at 34.29 27.94 0)
 			(hide yes)
