File: Output.kicad_sch (KiCad schematic)
At the start: 108 parts, among them J10 DB301V-3.5-3P-GN, J11 DB301V-3.5-3P-GN, J12 DB301V-3.5-3P-GN, J13 DB301V-3.5-3P-GN, J14 DB301V-3.5-3P-GN, J15 DB301V-3.5-3P-GN, J16 DB301V-3.5-3P-GN, J17 DB301V-3.5-3P-GN, J18 DB301V-3.5-3P-GN, J19 DB301V-3.5-3P-GN, J20 DB301V-3.5-3P-GN, J21 DB301V-3.5-3P-GN, J22 DB301V-3.5-3P-GN, J23 DB301V-3.5-3P-GN, J24 DB301V-3.5-3P-GN, J25 DB301V-3.5-3P-GN, J26 DB301V-3.5-3P-GN, J27 DB301V-3.5-3P-GN, J28 DB301V-3.5-3P-GN, J29 DB301V-3.5-3P-GN, J30 DB301V-3.5-3P-GN, J31 DB301V-3.5-3P-GN, J32 DB301V-3.5-3P-GN, J33 DB301V-3.5-3P-GN, J34 DB301V-3.5-3P-GN, J35 DB301V-3.5-3P-GN, J36 DB301V-3.5-3P-GN, J37 DB301V-3.5-3P-GN, J39 DB301V-3.5-3P-GN, J7 DB301V-3.5-3P-GN, J8 DB301V-3.5-3P-GN, J9 DB301V-3.5-3P-GN, U10 SN74LVC8T245PWR, U11 SN74LVC8T245PWR, U7 SN74LVC8T245PWR, U8 SN74LVC8T245PWR

Commit message: Start PCB layout and add mounting holes
Footprints placed on the board, H1-H4 mounting holes added to the
schematic, and schematic updates to Output and Power sheets.

Co-Authored-By: Claude Opus 5.5 <noreply@anthropic.com>
Connections:
- net +VIN_Z1: now also F10.1, F12.1, F14.1, F8.1; no longer F17.1, F19.1, F21.1, F23.1, F9.2, J8.1
- net +VIN_Z2: now also F17.1, F19.1, F21.1, F23.1; no longer F10.1, F12.1, F14.1, F8.1, F8.2, J7.1
- net +VIN_Z3: now also F24.1, F26.1, F28.1, F30.1; no longer F33.1, F35.1, F37.1, F39.1
- net +VIN_Z4: now also F33.1, F35.1, F37.1, F39.1; no longer F24.1, F26.1, F28.1, F30.1
- new net: F9.2, J8.1
- new net: F8.2, J7.1
