File: Output.kicad_sch (KiCad schematic)
At the start: 108 parts, among them J10 DB301V-3.5-3P-GN, J11 DB301V-3.5-3P-GN, J12 DB301V-3.5-3P-GN, J13 DB301V-3.5-3P-GN, J14 DB301V-3.5-3P-GN, J15 DB301V-3.5-3P-GN, J16 DB301V-3.5-3P-GN, J17 DB301V-3.5-3P-GN, J18 DB301V-3.5-3P-GN, J19 DB301V-3.5-3P-GN, J20 DB301V-3.5-3P-GN, J21 DB301V-3.5-3P-GN, J22 DB301V-3.5-3P-GN, J23 DB301V-3.5-3P-GN, J24 DB301V-3.5-3P-GN, J25 DB301V-3.5-3P-GN, J26 DB301V-3.5-3P-GN, J27 DB301V-3.5-3P-GN, J28 DB301V-3.5-3P-GN, J29 DB301V-3.5-3P-GN, J30 DB301V-3.5-3P-GN, J31 DB301V-3.5-3P-GN, J32 DB301V-3.5-3P-GN, J33 DB301V-3.5-3P-GN, J34 DB301V-3.5-3P-GN, J35 DB301V-3.5-3P-GN, J36 DB301V-3.5-3P-GN, J37 DB301V-3.5-3P-GN, J39 DB301V-3.5-3P-GN, J7 DB301V-3.5-3P-GN, J8 DB301V-3.5-3P-GN, J9 DB301V-3.5-3P-GN, U10 SN74LVC8T245PWR, U11 SN74LVC8T245PWR, U7 SN74LVC8T245PWR, U8 SN74LVC8T245PWR

Commit message: I think the output terminals are well-arranged now. Discovered pixel-blits layout all on my own.
Connections:
- net +VIN_Z1: now also F17.1, F19.1, F21.1, F23.1; no longer F10.1, F12.1, F14.1, F8.1
- net +VIN_Z2: now also F10.1, F12.1, F14.1, F8.1; no longer F17.1, F19.1, F21.1, F23.1
- net +VIN_Z3: now also F32.1, F33.1, F34.1, F35.1; no longer F28.1, F29.1, F30.1, F31.1
- net +VIN_Z4: now also F28.1, F29.1, F30.1, F31.1; no longer F32.1, F33.1, F34.1, F35.1
Changed lines of the file:
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@@
 			)
 		)
-		(property "Value" "+VIN_Z4"
+		(property "Value" "+VIN_Z3"
 			(at 237.236 106.426 0)
 			(show_name no)
@@
 			)
 		)
-		(property "Value" "+VIN_Z1"
+		(property "Value" "+VIN_Z2"
 			(at 53.086 94.996 0)
 			(show_name no)
@@
 			)
 		)
-		(property "Value" "+VIN_Z3"
+		(property "Value" "+VIN_Z4"
 			(at 178.816 139.446 0)
 			(show_name no)
@@
 			)
 		)
-		(property "Value" "+VIN_Z2"
+		(property "Value" "+VIN_Z1"
 			(at 116.586 106.426 0)
 			(show_name no)
@@
 			)
 		)
-		(property "Value" "+VIN_Z4"
+		(property "Value" "+VIN_Z3"
 			(at 237.236 94.996 0)
 			(show_name no)
@@
 			)
 		)
-		(property "Value" "+VIN_Z2"
+		(property "Value" "+VIN_Z1"
 			(at 116.586 129.286 0)
 			(show_name no)
@@
 			)
 		)
-		(property "Value" "+VIN_Z1"
+		(property "Value" "+VIN_Z2"
 			(at 53.086 140.716 0)
 			(show_name no)
@@
 			)
 		)
-		(property "Value" "+VIN_Z3"
+		(property "Value" "+VIN_Z4"
 			(at 178.816 150.876 0)
 			(show_name no)
@@
 			)
 		)
-		(property "Value" "+VIN_Z3"
+		(property "Value" "+VIN_Z4"
 			(at 178.816 128.016 0)
 			(show_name no)
@@
 			)
 		)
-		(property "Value" "+VIN_Z4"
+		(property "Value" "+VIN_Z3"
 			(at 237.236 83.566 0)
 			(show_name no)
@@
 			)
 		)
-		(property "Value" "+VIN_Z1"
+		(property "Value" "+VIN_Z2"
 			(at 53.086 117.856 0)
 			(show_name no)
@@
 			)
 		)
-		(property "Value" "+VIN_Z2"
+		(property "Value" "+VIN_Z1"
 			(at 116.586 83.566 0)
 			(show_name no)
@@
 			)
 		)
-		(property "Value" "+VIN_Z4"
+		(property "Value" "+VIN_Z3"
 			(at 237.236 72.136 0)
 			(show_name no)
@@
 			)
 		)
-		(property "Value" "+VIN_Z3"
+		(property "Value" "+VIN_Z4"
 			(at 178.816 116.586 0)
 			(show_name no)
@@
 			)
 		)
-		(property "Value" "+VIN_Z2"
+		(property "Value" "+VIN_Z1"
 			(at 116.586 152.146 0)
 			(show_name no)
@@
 			)
 		)
-		(property "Value" "+VIN_Z1"
+		(property "Value" "+VIN_Z2"
 			(at 48.26 72.644 0)
 			(show_name no)

Commit message: Some changes, not sure what...
Connections:
- net +VIN_Z3: now also F28.1, F30.1, F36.1, F38.1; no longer F25.1, F27.1, F33.1, F35.1
- net +VIN_Z4: now also F25.1, F27.1, F33.1, F35.1; no longer F28.1, F30.1, F36.1, F38.1
Changed lines of the file:
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@@
 			)
 		)
-		(property "Value" "+VIN_Z3"
+		(property "Value" "+VIN_Z4"
 			(at 178.816 82.296 0)
 			(show_name no)
@@
 			)
 		)
-		(property "Value" "+VIN_Z3"
+		(property "Value" "+VIN_Z4"
 			(at 237.236 106.426 0)
 			(show_name no)
@@
 			)
 		)
-		(property "Value" "+VIN_Z4"
+		(property "Value" "+VIN_Z3"
 			(at 178.816 139.446 0)
 			(show_name no)
@@
 			)
 		)
-		(property "Value" "+VIN_Z4"
+		(property "Value" "+VIN_Z3"
 			(at 237.236 117.856 0)
 			(show_name no)
@@
 			)
 		)
-		(property "Value" "+VIN_Z3"
+		(property "Value" "+VIN_Z4"
 			(at 237.236 83.566 0)
 			(show_name no)
@@
 			)
 		)
-		(property "Value" "+VIN_Z4"
+		(property "Value" "+VIN_Z3"
 			(at 237.236 140.716 0)
 			(show_name no)
@@
 			)
 		)
-		(property "Value" "+VIN_Z4"
+		(property "Value" "+VIN_Z3"
 			(at 178.816 116.586 0)
 			(show_name no)
@@
 			)
 		)
-		(property "Value" "+VIN_Z3"
+		(property "Value" "+VIN_Z4"
 			(at 178.816 105.156 0)
 			(show_name no)
