File: universal-strip-controller.kicad_pcb (KiCad board)
At the start: 2 copper layers, 181 x 125 mm, 0 parts

Commit message: Seems messed up?
Parts:
- added BT1: CR1220, KiCad_Standard:Battery_Panasonic_CR1220-VCN_Vertical_CircularHoles, F.Cu at (-4.87, 218.5)
- added C10: 100n, RPI_COMPILED:generic_capc1005x50, F.Cu at (30.5, 183.3)
- added C11: 100n, RPI_COMPILED:generic_capc1005x50, F.Cu at (30.5, 184.8)
- added C118: 1uF, PixelBlit:C_0402, F.Cu at (1.94, 224.6)
- added C119: 100n, RPI_COMPILED:generic_capc1005x50, F.Cu at (-95.1, 215.6)
- added C12: 100n, RPI_COMPILED:generic_capc1005x50, F.Cu at (30.5, 186.4)
- added C120: 100n, RPI_COMPILED:generic_capc1005x50, F.Cu at (-95.1, 217.2)
- added C121: 100n, RPI_COMPILED:generic_capc1005x50, F.Cu at (-95.1, 218.7)
- added C122: 100n, RPI_COMPILED:generic_capc1005x50, F.Cu at (-95.1, 220.3)
- added C123: 100n, RPI_COMPILED:generic_capc1005x50, F.Cu at (-95.1, 221.8)
- added C124: 100n, RPI_COMPILED:generic_capc1005x50, F.Cu at (-92.6, 215.6)
- added C125: 100n, RPI_COMPILED:generic_capc1005x50, F.Cu at (-92.6, 217.2)
- added C126: 100n, RPI_COMPILED:generic_capc1005x50, F.Cu at (-92.6, 218.7)
- added C127: 100n, RPI_COMPILED:generic_capc1005x50, F.Cu at (-92.6, 220.3)
- added C128: 100n, RPI_COMPILED:generic_capc1005x50, F.Cu at (-92.6, 221.8)
- added C129: 100n, RPI_COMPILED:generic_capc1005x50, F.Cu at (-90.1, 215.6)
- added C13: 100n, RPI_COMPILED:generic_capc1005x50, F.Cu at (30.5, 187.9)
- added C130: 100n, RPI_COMPILED:generic_capc1005x50, F.Cu at (-90.1, 217.2)
- added C131: 100n, RPI_COMPILED:generic_capc1005x50, F.Cu at (-90.1, 218.7)
- added C132: 100n, RPI_COMPILED:generic_capc1005x50, F.Cu at (-90.1, 220.3)
- added C133: 100n, RPI_COMPILED:generic_capc1005x50, F.Cu at (44.9, 167.4)
- added C134: 100n, RPI_COMPILED:generic_capc1005x50, F.Cu at (44.9, 168.9)
- added C135: 100n, RPI_COMPILED:generic_capc1005x50, F.Cu at (44.9, 170.5)
- added C136: 100n, RPI_COMPILED:generic_capc1005x50, F.Cu at (44.9, 172.0)
- added C137: 100n, RPI_COMPILED:generic_capc1005x50, F.Cu at (44.9, 173.6)
- added C138: 100n, RPI_COMPILED:generic_capc1005x50, F.Cu at (44.9, 175.1)
- added C139: 100n, RPI_COMPILED:generic_capc1005x50, F.Cu at (44.9, 176.7)
- added C14: 100n, RPI_COMPILED:generic_capc1005x50, F.Cu at (30.5, 189.5)
- added C140: 100n, RPI_COMPILED:generic_capc1005x50, F.Cu at (44.9, 178.2)
- added C15: 100n, RPI_COMPILED:generic_capc1005x50, F.Cu at (30.5, 191.0)
- added C16: 100n, RPI_COMPILED:generic_capc1005x50, F.Cu at (30.5, 192.6)
- added C17: 100n, RPI_COMPILED:generic_capc1005x50, F.Cu at (33.0, 183.3)
- added C18: 100n, RPI_COMPILED:generic_capc1005x50, F.Cu at (33.0, 184.8)
- added C19: 10u, RPI_COMPILED:generic_capc2012x125, F.Cu at (33.2, 213.0)
- added C2: 100n, RPI_COMPILED:generic_capc1005x50, F.Cu at (28.0, 183.3)
- added C20: 100n, RPI_COMPILED:generic_capc1005x50, F.Cu at (33.0, 186.4)
- added C21: 100n, RPI_COMPILED:generic_capc1005x50, F.Cu at (33.0, 187.9)
- added C23: 22uF, PixelBlit:C_0805, F.Cu at (42.8, 149.9)
- added C24: 22uF, PixelBlit:C_0805, F.Cu at (42.8, 153.0)
- added C25: 10uF, PixelBlit:C_0603, F.Cu at (41.7, 167.7)
- added C26: 10uF, PixelBlit:C_0603, F.Cu at (41.7, 170.0)
- added C27: 100nF, PixelBlit:C_0603, F.Cu at (41.7, 172.2)
- added C28: 100nF, PixelBlit:C_0402, F.Cu at (27.2, 177.9)
- added C29: 10uF, PixelBlit:C_0603, F.Cu at (41.7, 174.5)
- added C3: 15p, RPI_COMPILED:generic_capc1005x50, F.Cu at (28.0, 184.8)
- added C30: 100nF, PixelBlit:C_0603, F.Cu at (41.7, 176.7)
- added C31: 10uF, PixelBlit:C_0603, F.Cu at (41.7, 179.0)
- added C32: 10uF, PixelBlit:C_0805, F.Cu at (42.8, 156.0)
- added C33: 47uF, PixelBlit:C_0805, F.Cu at (42.8, 159.1)
- added C34: 100nF, PixelBlit:C_0402, F.Cu at (-22.8, 158.5)
- added C35: 100nF, PixelBlit:C_0402, F.Cu at (-22.8, 160.4)
- added C36: 100nF, PixelBlit:C_0402, F.Cu at (-22.8, 162.2)
- added C37: 100nF, PixelBlit:C_0402, F.Cu at (-22.8, 164.1)
- added C38: 100nF, PixelBlit:C_0402, F.Cu at (-22.8, 165.9)
- added C39: 100nF, PixelBlit:C_0402, F.Cu at (-22.8, 167.8)
- added C4: 15p, RPI_COMPILED:generic_capc1005x50, F.Cu at (28.0, 186.4)
- added C40: 100nF, PixelBlit:C_0402, F.Cu at (-22.8, 169.6)
- added C41: 100nF, PixelBlit:C_0402, F.Cu at (-22.8, 171.5)
- added C6: 4.7u, RPI_COMPILED:generic_capc1005x50_wide, F.Cu at (28.0, 187.9)
- added C7: 4.7u, RPI_COMPILED:generic_capc1005x50_wide, F.Cu at (28.0, 189.5)
- added C8: 100n, RPI_COMPILED:generic_capc1005x50, F.Cu at (28.0, 191.0)
- added C9: 4.7u, RPI_COMPILED:generic_capc1005x50, F.Cu at (28.0, 192.6)
- added D1: B5819W, PixelBlit:D_SOD-123, F.Cu at (34.2, 210.1)
- added D10: BZT52C15V, Diode_SMD:D_SOD-123, F.Cu at (28.6, 175.3)
- added D11: SK6812MINI, LED_SMD:LED_SK6812MINI_PLCC4_3.5x3.5mm_P1.75mm, F.Cu at (-93.0, 207.2)
- added D12: SK6812MINI, LED_SMD:LED_SK6812MINI_PLCC4_3.5x3.5mm_P1.75mm, F.Cu at (-93.0, 212.3)
- added D13: SK6812MINI, LED_SMD:LED_SK6812MINI_PLCC4_3.5x3.5mm_P1.75mm, F.Cu at (-86.3, 196.9)
- added D14: SK6812MINI, LED_SMD:LED_SK6812MINI_PLCC4_3.5x3.5mm_P1.75mm, F.Cu at (-86.3, 202.0)
- added D15: SK6812MINI, LED_SMD:LED_SK6812MINI_PLCC4_3.5x3.5mm_P1.75mm, F.Cu at (-86.3, 207.2)
- added D16: SK6812MINI, LED_SMD:LED_SK6812MINI_PLCC4_3.5x3.5mm_P1.75mm, F.Cu at (-86.3, 212.3)
- added D17: SK6812MINI, LED_SMD:LED_SK6812MINI_PLCC4_3.5x3.5mm_P1.75mm, F.Cu at (-79.6, 196.9)
- added D18: SK6812MINI, LED_SMD:LED_SK6812MINI_PLCC4_3.5x3.5mm_P1.75mm, F.Cu at (-79.6, 202.0)
- added D19: SK6812MINI, LED_SMD:LED_SK6812MINI_PLCC4_3.5x3.5mm_P1.75mm, F.Cu at (-79.6, 207.2)
- added D2: USBLC6-2SC6, PixelBlit:SOT-23-6_L2.9-W1.6-P0.95-LS2.8-BL, F.Cu at (29.2, 211.9)
- added D20: SK6812MINI, LED_SMD:LED_SK6812MINI_PLCC4_3.5x3.5mm_P1.75mm, F.Cu at (-79.6, 212.3)
- added D21: SK6812MINI, LED_SMD:LED_SK6812MINI_PLCC4_3.5x3.5mm_P1.75mm, F.Cu at (-72.9, 196.9)
- added D22: SK6812MINI, LED_SMD:LED_SK6812MINI_PLCC4_3.5x3.5mm_P1.75mm, F.Cu at (-72.9, 202.0)
- added D23: SK6812MINI, LED_SMD:LED_SK6812MINI_PLCC4_3.5x3.5mm_P1.75mm, F.Cu at (-72.9, 207.2)
- added D24: SK6812MINI, LED_SMD:LED_SK6812MINI_PLCC4_3.5x3.5mm_P1.75mm, F.Cu at (-72.9, 212.3)
- added D3: SK6812MINI, LED_SMD:LED_SK6812MINI_PLCC4_3.5x3.5mm_P1.75mm, F.Cu at (-93.0, 196.9)
- added D4: B5819W, PixelBlit:D_SOD-123, F.Cu at (28.7, 172.0)
- added D5: SS34, PCM_JLCPCB:D_SMA, F.Cu at (36.6, 150.7)
- added D6: SS34, PCM_JLCPCB:D_SMA, F.Cu at (36.6, 155.2)
- added D7: SS34, PCM_JLCPCB:D_SMA, F.Cu at (36.6, 159.8)
- added D8: SS34, PCM_JLCPCB:D_SMA, F.Cu at (36.6, 164.3)
- added D9: SK6812MINI, LED_SMD:LED_SK6812MINI_PLCC4_3.5x3.5mm_P1.75mm, F.Cu at (-93.0, 202.0)
- added F1: 3557-2, EasyEDA:FUSE-TH_4P-L19.8-W6.7_3557-2, F.Cu at (21.9, 114.7)
- added F10: 1812L400/16GR, EasyEDA:F1812, F.Cu at (-41.0, 123.7)
- added F11: 1812L400/16GR, EasyEDA:F1812, F.Cu at (-41.0, 128.9)
- added F12: 1812L400/16GR, EasyEDA:F1812, F.Cu at (-41.0, 134.2)
- added F13: 1812L400/16GR, EasyEDA:F1812, F.Cu at (-41.0, 139.4)
- added F14: 1812L400/16GR, EasyEDA:F1812, F.Cu at (-41.0, 144.6)
- added F15: 1812L400/16GR, EasyEDA:F1812, F.Cu at (-41.0, 149.8)
- added F16: 1812L400/16GR, EasyEDA:F1812, F.Cu at (-41.0, 155.0)
- added F17: 1812L400/16GR, EasyEDA:F1812, F.Cu at (-32.8, 113.3)
- added F18: 1812L400/16GR, EasyEDA:F1812, F.Cu at (-32.8, 118.5)
- added F19: 1812L400/16GR, EasyEDA:F1812, F.Cu at (-32.8, 123.7)
- added F2: 3557-2, EasyEDA:FUSE-TH_4P-L19.8-W6.7_3557-2, F.Cu at (21.9, 122.7)
- added F20: 1812L400/16GR, EasyEDA:F1812, F.Cu at (-32.8, 128.9)
- added F21: 1812L400/16GR, EasyEDA:F1812, F.Cu at (-32.8, 134.2)
- added F22: 1812L400/16GR, EasyEDA:F1812, F.Cu at (-32.8, 139.4)
- added F23: 1812L400/16GR, EasyEDA:F1812, F.Cu at (-32.8, 144.6)
- added F24: 1812L400/16GR, EasyEDA:F1812, F.Cu at (-32.8, 149.8)
- added F25: 1812L400/16GR, EasyEDA:F1812, F.Cu at (-32.8, 155.0)
- added F26: 1812L400/16GR, EasyEDA:F1812, F.Cu at (-24.6, 113.3)
- added F27: 1812L400/16GR, EasyEDA:F1812, F.Cu at (-24.6, 118.5)
- added F28: 1812L400/16GR, EasyEDA:F1812, F.Cu at (-24.6, 123.7)
- added F29: 1812L400/16GR, EasyEDA:F1812, F.Cu at (-24.6, 128.9)
- added F3: 3557-2, EasyEDA:FUSE-TH_4P-L19.8-W6.7_3557-2, F.Cu at (21.9, 130.7)
- added F30: 1812L400/16GR, EasyEDA:F1812, F.Cu at (-24.6, 134.2)
- added F31: 1812L400/16GR, EasyEDA:F1812, F.Cu at (-24.6, 139.4)
- added F32: 1812L400/16GR, EasyEDA:F1812, F.Cu at (-24.6, 144.6)
- added F33: 1812L400/16GR, EasyEDA:F1812, F.Cu at (-24.6, 149.8)
- added F34: 1812L400/16GR, EasyEDA:F1812, F.Cu at (-24.6, 155.0)
- added F35: 1812L400/16GR, EasyEDA:F1812, F.Cu at (-16.4, 113.3)
- added F36: 1812L400/16GR, EasyEDA:F1812, F.Cu at (-16.4, 118.5)
- added F37: 1812L400/16GR, EasyEDA:F1812, F.Cu at (-16.4, 123.7)
- added F38: 1812L400/16GR, EasyEDA:F1812, F.Cu at (-16.4, 128.9)
- added F39: 1812L400/16GR, EasyEDA:F1812, F.Cu at (-16.4, 134.2)
- added F4: 3557-2, EasyEDA:FUSE-TH_4P-L19.8-W6.7_3557-2, F.Cu at (21.9, 138.7)
- added F5: 3557-2, EasyEDA:FUSE-TH_4P-L19.8-W6.7_3557-2, F.Cu at (21.9, 146.6)
- added F6: 3557-2, EasyEDA:FUSE-TH_4P-L19.8-W6.7_3557-2, F.Cu at (21.9, 154.6)
- added F7: 3557-2, EasyEDA:FUSE-TH_4P-L19.8-W6.7_3557-2, F.Cu at (21.9, 162.6)
- added F8: 1812L400/16GR, EasyEDA:F1812, F.Cu at (-41.0, 113.3)
- added F9: 1812L400/16GR, EasyEDA:F1812, F.Cu at (-41.0, 118.5)
- added J1: Conn_01x03_Pin, Connector_PinHeader_2.54mm:PinHeader_1x03_P2.54mm_Vertical, F.Cu at (29.0, 202.3)
- added J10: DB301V-3.5-3P-GN, PixelBlit:CONN-TH_DB301V-3.5-3P-GN, F.Cu at (-89.9, 138.2)
- added J11: DB301V-3.5-3P-GN, PixelBlit:CONN-TH_DB301V-3.5-3P-GN, F.Cu at (-89.9, 146.0)
- added J12: DB301V-3.5-3P-GN, PixelBlit:CONN-TH_DB301V-3.5-3P-GN, F.Cu at (-89.9, 153.8)
- added J13: DB301V-3.5-3P-GN, PixelBlit:CONN-TH_DB301V-3.5-3P-GN, F.Cu at (-89.9, 161.6)
- added J14: DB301V-3.5-3P-GN, PixelBlit:CONN-TH_DB301V-3.5-3P-GN, F.Cu at (-89.9, 169.4)
- added J15: DB301V-3.5-3P-GN, PixelBlit:CONN-TH_DB301V-3.5-3P-GN, F.Cu at (-89.9, 177.3)
- added J16: DB301V-3.5-3P-GN, PixelBlit:CONN-TH_DB301V-3.5-3P-GN, F.Cu at (-77.1, 114.7)
- added J17: DB301V-3.5-3P-GN, PixelBlit:CONN-TH_DB301V-3.5-3P-GN, F.Cu at (-77.1, 122.6)
- added J18: DB301V-3.5-3P-GN, PixelBlit:CONN-TH_DB301V-3.5-3P-GN, F.Cu at (-77.1, 130.4)
- added J19: DB301V-3.5-3P-GN, PixelBlit:CONN-TH_DB301V-3.5-3P-GN, F.Cu at (-77.1, 138.2)
- added J2: Conn_01x02_Pin, Connector_PinHeader_2.54mm:PinHeader_1x02_P2.54mm_Vertical, F.Cu at (34.5, 216.9)
- added J20: DB301V-3.5-3P-GN, PixelBlit:CONN-TH_DB301V-3.5-3P-GN, F.Cu at (-77.1, 146.0)
- added J21: DB301V-3.5-3P-GN, PixelBlit:CONN-TH_DB301V-3.5-3P-GN, F.Cu at (-77.1, 153.8)
- added J22: DB301V-3.5-3P-GN, PixelBlit:CONN-TH_DB301V-3.5-3P-GN, F.Cu at (-77.1, 161.6)
- added J23: DB301V-3.5-3P-GN, PixelBlit:CONN-TH_DB301V-3.5-3P-GN, F.Cu at (-77.1, 169.4)
- added J24: DB301V-3.5-3P-GN, PixelBlit:CONN-TH_DB301V-3.5-3P-GN, F.Cu at (-77.1, 177.3)
- added J25: DB301V-3.5-3P-GN, PixelBlit:CONN-TH_DB301V-3.5-3P-GN, F.Cu at (-64.3, 114.7)
- added J26: DB301V-3.5-3P-GN, PixelBlit:CONN-TH_DB301V-3.5-3P-GN, F.Cu at (-64.3, 122.6)
- added J27: DB301V-3.5-3P-GN, PixelBlit:CONN-TH_DB301V-3.5-3P-GN, F.Cu at (-64.3, 130.4)
- added J28: DB301V-3.5-3P-GN, PixelBlit:CONN-TH_DB301V-3.5-3P-GN, F.Cu at (-64.3, 138.2)
- added J29: DB301V-3.5-3P-GN, PixelBlit:CONN-TH_DB301V-3.5-3P-GN, F.Cu at (-64.3, 146.0)
- added J3: DBT50G-9.5-2P, EasyEDA:CONN-TH_2P-P9.50_DBT50G-9.5-2P, F.Cu at (226.5, 137.7)
- added J30: DB301V-3.5-3P-GN, PixelBlit:CONN-TH_DB301V-3.5-3P-GN, F.Cu at (-64.3, 153.8)
- added J31: DB301V-3.5-3P-GN, PixelBlit:CONN-TH_DB301V-3.5-3P-GN, F.Cu at (-64.3, 161.6)
- added J32: DB301V-3.5-3P-GN, PixelBlit:CONN-TH_DB301V-3.5-3P-GN, F.Cu at (-64.3, 169.4)
- added J33: DB301V-3.5-3P-GN, PixelBlit:CONN-TH_DB301V-3.5-3P-GN, F.Cu at (-64.3, 177.3)
- added J34: DB301V-3.5-3P-GN, PixelBlit:CONN-TH_DB301V-3.5-3P-GN, F.Cu at (-51.5, 114.7)
- added J35: DB301V-3.5-3P-GN, PixelBlit:CONN-TH_DB301V-3.5-3P-GN, F.Cu at (-51.5, 122.6)
- added J36: DB301V-3.5-3P-GN, PixelBlit:CONN-TH_DB301V-3.5-3P-GN, F.Cu at (-51.5, 130.4)
- added J37: DB301V-3.5-3P-GN, PixelBlit:CONN-TH_DB301V-3.5-3P-GN, F.Cu at (-51.5, 138.2)
- added J38: 2.54-1*4, PixelBlit:HDR-TH_4P-P2.54-V-M-1, F.Cu at (17.1, 168.4)
- added J39: DB301V-3.5-3P-GN, PixelBlit:CONN-TH_DB301V-3.5-3P-GN, F.Cu at (-51.5, 146.0)
- added J4: DBT50G-9.5-2P, EasyEDA:CONN-TH_2P-P9.50_DBT50G-9.5-2P, F.Cu at (214.0, 74.2)
- added J5: DBT50G-9.5-2P, EasyEDA:CONN-TH_2P-P9.50_DBT50G-9.5-2P, F.Cu at (0.55, 150.5)
- added J6: DBT50G-9.5-2P, EasyEDA:CONN-TH_2P-P9.50_DBT50G-9.5-2P, F.Cu at (0.55, 168.0)
- added J7: DB301V-3.5-3P-GN, PixelBlit:CONN-TH_DB301V-3.5-3P-GN, F.Cu at (-89.9, 114.7)
- added J8: DB301V-3.5-3P-GN, PixelBlit:CONN-TH_DB301V-3.5-3P-GN, F.Cu at (-89.9, 122.6)
- added J9: DB301V-3.5-3P-GN, PixelBlit:CONN-TH_DB301V-3.5-3P-GN, F.Cu at (-89.9, 130.4)
- added L1: 3.3u, RPI_COMPILED:abracon_aota-b201610s3r3-101-t, F.Cu at (34.2, 227.0)
- added L2: FXL0420-1R5-M, EasyEDA:IND-SMD_L4.4-W4.2, F.Cu at (19.1, 173.1)
- added PWR_LED1: Red, PixelBlit:D_0603, F.Cu at (13.5, 171.6)
- added PWR_LED2: Red, PixelBlit:D_0603, F.Cu at (13.5, 174.2)
- added PWR_LED3: Red, PixelBlit:D_0603, F.Cu at (13.5, 176.8)
- added R1: 10k, RPI_COMPILED:generic_resc1005x35, F.Cu at (33.0, 189.5)
- added R10: 0, RPI_COMPILED:generic_resc1005x35, F.Cu at (35.5, 191.0)
- added R100: 10kΩ, PixelBlit:R_0603, F.Cu at (34.3, 176.7)
- added R101: 10kΩ, PixelBlit:R_0603, F.Cu at (34.3, 179.0)
- added R102: 10kΩ, PixelBlit:R_0603, F.Cu at (38.0, 167.7)
- added R103: 10kΩ, PixelBlit:R_0603, F.Cu at (38.0, 170.0)
- added R104: 10kΩ, PixelBlit:R_0603, F.Cu at (38.0, 172.2)
- added R105: 10kΩ, PixelBlit:R_0603, F.Cu at (38.0, 174.5)
- added R106: 10kΩ, PixelBlit:R_0603, F.Cu at (38.0, 176.7)
- added R11: 5.1kΩ, PixelBlit:R_0402, F.Cu at (1.94, 220.8)
- added R12: 5.1kΩ, PixelBlit:R_0402, F.Cu at (1.94, 222.7)
- added R13: 10kΩ, PixelBlit:R_0603, F.Cu at (34.3, 167.7)
- added R14: 560kΩ, PixelBlit:R_0402, F.Cu at (41.2, 131.0)
- added R15: 100kΩ, PixelBlit:R_0402, F.Cu at (41.2, 132.9)
- added R16: 100kΩ, PixelBlit:R_0603, F.Cu at (34.3, 170.0)
- added R17: 100kΩ, PixelBlit:R_0603, F.Cu at (34.3, 172.2)
- added R18: 1kΩ, PixelBlit:R_0402, F.Cu at (41.2, 134.7)
- added R19: 47Ω, PixelBlit:R_0402, F.Cu at (-87.5, 220.4)
- added R2: 1k, RPI_COMPILED:generic_resc1005x35, F.Cu at (33.0, 191.0)
- added R20: 2.2kΩ, Resistor_SMD:R_0603_1608Metric, F.Cu at (41.8, 145.0)
- added R21: 47Ω, PixelBlit:R_0402, F.Cu at (-34.2, 158.5)
- added R22: 2mΩ, Resistor_SMD:R_Shunt_Vishay_WSK2512_6332Metric_T1.19mm, F.Cu at (37.4, 113.1)
- added R23: 10Ω, PixelBlit:R_0402, F.Cu at (41.2, 136.6)
- added R24: 47Ω, PixelBlit:R_0402, F.Cu at (-34.2, 160.4)
- added R25: 47Ω, PixelBlit:R_0402, F.Cu at (-34.2, 162.2)
- added R26: 47Ω, PixelBlit:R_0402, F.Cu at (-34.2, 164.1)
- added R27: 47Ω, PixelBlit:R_0402, F.Cu at (-34.2, 165.9)
- added R28: 47Ω, PixelBlit:R_0402, F.Cu at (-34.2, 167.8)
- added R29: 47Ω, PixelBlit:R_0402, F.Cu at (-34.2, 169.6)
- added R3: 33, RPI_COMPILED:generic_resc1005x35, F.Cu at (33.0, 192.6)
- added R30: 47Ω, PixelBlit:R_0402, F.Cu at (-34.2, 171.5)
- added R31: 47Ω, PixelBlit:R_0402, F.Cu at (-34.2, 173.3)
- added R32: 47Ω, PixelBlit:R_0402, F.Cu at (-31.3, 158.5)
- added R33: 47Ω, PixelBlit:R_0402, F.Cu at (-31.3, 160.4)
- added R34: 47Ω, PixelBlit:R_0402, F.Cu at (-31.3, 162.2)
- added R35: 47Ω, PixelBlit:R_0402, F.Cu at (-31.3, 164.1)
- added R36: 47Ω, PixelBlit:R_0402, F.Cu at (-31.3, 165.9)
- added R37: 47Ω, PixelBlit:R_0402, F.Cu at (-31.3, 167.8)
- added R38: 47Ω, PixelBlit:R_0402, F.Cu at (-31.3, 169.6)
- added R39: 47Ω, PixelBlit:R_0402, F.Cu at (-31.3, 171.5)
- added R4: 1k, RPI_COMPILED:generic_resc1005x35, F.Cu at (35.5, 183.3)
- added R40: 47Ω, PixelBlit:R_0402, F.Cu at (-31.3, 173.3)
- added R41: 47Ω, PixelBlit:R_0402, F.Cu at (-28.5, 158.5)
- added R42: 47Ω, PixelBlit:R_0402, F.Cu at (-28.5, 160.4)
- added R43: 47Ω, PixelBlit:R_0402, F.Cu at (-28.5, 162.2)
- added R44: 47Ω, PixelBlit:R_0402, F.Cu at (-28.5, 164.1)
- added R45: 47Ω, PixelBlit:R_0402, F.Cu at (-28.5, 165.9)
- added R46: 47Ω, PixelBlit:R_0402, F.Cu at (-28.5, 167.8)
- added R47: 47Ω, PixelBlit:R_0402, F.Cu at (-28.5, 169.6)
- added R48: 47Ω, PixelBlit:R_0402, F.Cu at (-28.5, 171.5)
- added R49: 47Ω, PixelBlit:R_0402, F.Cu at (-28.5, 173.3)
- added R5: 8.2kΩ, Resistor_SMD:R_0603_1608Metric, F.Cu at (41.8, 142.5)
- added R50: 47Ω, PixelBlit:R_0402, F.Cu at (-25.6, 158.5)
- added R51: 47Ω, PixelBlit:R_0402, F.Cu at (-25.6, 160.4)
- added R52: 47Ω, PixelBlit:R_0402, F.Cu at (-25.6, 162.2)
- added R53: 47Ω, PixelBlit:R_0402, F.Cu at (-25.6, 164.1)
- added R54: 47Ω, PixelBlit:R_0402, F.Cu at (-25.6, 165.9)
- added R55: 10Ω, PixelBlit:R_0402, F.Cu at (41.2, 138.4)
- added R56: 2mΩ, Resistor_SMD:R_Shunt_Vishay_WSK2512_6332Metric_T1.19mm, F.Cu at (37.4, 118.0)
- added R57: 10Ω, PixelBlit:R_0402, F.Cu at (41.2, 140.3)
- added R58: 10Ω, PixelBlit:R_0402, F.Cu at (44.1, 131.0)
- added R59: 2mΩ, Resistor_SMD:R_Shunt_Vishay_WSK2512_6332Metric_T1.19mm, F.Cu at (37.4, 122.8)
- added R6: 1k, RPI_COMPILED:generic_resc1005x35, F.Cu at (35.5, 184.8)
- added R60: 10Ω, PixelBlit:R_0402, F.Cu at (44.1, 132.9)
- added R61: 10Ω, PixelBlit:R_0402, F.Cu at (44.1, 134.7)
- added R62: 2mΩ, Resistor_SMD:R_Shunt_Vishay_WSK2512_6332Metric_T1.19mm, F.Cu at (37.4, 127.7)
- added R63: 10Ω, PixelBlit:R_0402, F.Cu at (44.1, 136.6)
- added R64: 10Ω, PixelBlit:R_0402, F.Cu at (44.1, 138.4)
- added R7: 27, RPI_COMPILED:generic_resc1005x35, F.Cu at (35.5, 186.4)
- added R8: 27, RPI_COMPILED:generic_resc1005x35, F.Cu at (35.5, 187.9)
- added R9: 0, RPI_COMPILED:generic_resc1005x35, F.Cu at (35.5, 189.5)
- added R94: 10kΩ, PixelBlit:R_0603, F.Cu at (30.4, 215.7)
- added R95: 10kΩ, PixelBlit:R_0603, F.Cu at (30.4, 217.9)
- added R96: 10kΩ, PixelBlit:R_0603, F.Cu at (30.4, 220.2)
- added R97: 10kΩ, PixelBlit:R_0603, F.Cu at (30.4, 222.4)
- added R98: 470Ω, PixelBlit:R_0603, F.Cu at (30.4, 224.7)
- added R99: 10kΩ, PixelBlit:R_0603, F.Cu at (34.3, 174.5)
- added SW1: 434133025816, RPI_COMPILED:wurthelek_434133025816, F.Cu at (34.2, 202.1)
- added SW2: 434133025816, RPI_COMPILED:wurthelek_434133025816, F.Cu at (34.2, 206.3)
- added TP2: TestPoint, PixelBlit:TestPoint_Pad_1.0x1.0mm, F.Cu at (24.2, 171.8)
- added TP3: TestPoint, PixelBlit:TestPoint_Pad_1.0x1.0mm, F.Cu at (24.2, 174.9)
- added U1: RP2350B, RPI_COMPILED:rpi_rp2350b_vias, F.Cu at (22.7, 220.6)
- added U10: SN74LVC8T245PWR, PixelBlit:TSSOP-24_L7.8-W4.4-P0.65-LS6.4-BL, F.Cu at (-40.2, 179.3)
- added U11: SN74LVC8T245PWR, PixelBlit:TSSOP-24_L7.8-W4.4-P0.65-LS6.4-BL, F.Cu at (-40.2, 188.0)
- added U12: INA226, Package_SO:TSSOP-10_3x3mm_P0.5mm, F.Cu at (36.1, 132.4)
- added U13: INA226, Package_SO:TSSOP-10_3x3mm_P0.5mm, F.Cu at (36.1, 137.0)
- added U14: INA226, Package_SO:TSSOP-10_3x3mm_P0.5mm, F.Cu at (36.1, 141.6)
- added U15: INA226, Package_SO:TSSOP-10_3x3mm_P0.5mm, F.Cu at (36.1, 146.1)
- added U2: RPI RM2, RF_Module:RMC20452T, F.Cu at (8.20, 205.0)
- added U3: W25Q128JVSIQ, RPI_COMPILED:generic_soic127p790x195-8, F.Cu at (31.7, 196.9)
- added U4: SN74LVC1T45DBV, Package_TO_SOT_SMD:SOT-23-6, F.Cu at (-86.3, 217.2)
- added U5: TPS63070RNMR, PixelBlit:VQFN-HR-15_L3.0-W2.5-P0.50-BL_TPS63070RNMR, F.Cu at (42.9, 162.9)
- added U6: ~, PixelBlit:SOT-23-5_L3.0-W1.7-P0.95-LS2.8-BR, F.Cu at (17.8, 177.9)
- added U7: SN74LVC8T245PWR, PixelBlit:TSSOP-24_L7.8-W4.4-P0.65-LS6.4-BL, F.Cu at (-40.2, 161.9)
- added U8: SN74LVC8T245PWR, PixelBlit:TSSOP-24_L7.8-W4.4-P0.65-LS6.4-BL, F.Cu at (-40.2, 170.6)
- added U9: DS3231SN, Package_SO:SOIC-16W_7.5x10.3mm_P1.27mm, F.Cu at (10.3, 220.6)
- added USB1: TYPE-C 16PIN 2MD(073), PixelBlit:USB-C-SMD_TYPE-C-6PIN-2MD-073, F.Cu at (-4.91, 223.4)
- added X1: 12MHz, RPI_COMPILED:generic_xtalcc320x250x80-4, F.Cu at (35.0, 223.7)
