File: universal-strip-controller.kicad_pcb (KiCad board)
At the start: 2 copper layers, 181 x 125 mm, 0 parts

Commit message: Start PCB layout and add mounting holes
Footprints placed on the board, H1-H4 mounting holes added to the
schematic, and schematic updates to Output and Power sheets.

Co-Authored-By: Claude Opus 5.5 <noreply@anthropic.com>
Parts:
- added BT1: CR1220, KiCad_Standard:Battery_Panasonic_CR1220-VCN_Vertical_CircularHoles, F.Cu at (-59.5, 158.8)
- added C10: 100n, RPI_COMPILED:generic_capc1005x50, F.Cu at (-24.1, 123.6)
- added C11: 100n, RPI_COMPILED:generic_capc1005x50, F.Cu at (-24.1, 125.1)
- added C118: 1uF, PixelBlit:C_0402, F.Cu at (-52.7, 164.8)
- added C119: 100n, RPI_COMPILED:generic_capc1005x50, F.Cu at (-149.8, 155.9)
- added C12: 100n, RPI_COMPILED:generic_capc1005x50, F.Cu at (-24.1, 126.7)
- added C120: 100n, RPI_COMPILED:generic_capc1005x50, F.Cu at (-149.8, 157.5)
- added C121: 100n, RPI_COMPILED:generic_capc1005x50, F.Cu at (-149.8, 159.0)
- added C122: 100n, RPI_COMPILED:generic_capc1005x50, F.Cu at (-149.8, 160.6)
- added C123: 100n, RPI_COMPILED:generic_capc1005x50, F.Cu at (-149.8, 162.1)
- added C124: 100n, RPI_COMPILED:generic_capc1005x50, F.Cu at (-147.2, 155.9)
- added C125: 100n, RPI_COMPILED:generic_capc1005x50, F.Cu at (-147.2, 157.5)
- added C126: 100n, RPI_COMPILED:generic_capc1005x50, F.Cu at (-147.2, 159.0)
- added C127: 100n, RPI_COMPILED:generic_capc1005x50, F.Cu at (-147.2, 160.6)
- added C128: 100n, RPI_COMPILED:generic_capc1005x50, F.Cu at (-147.2, 162.1)
- added C129: 100n, RPI_COMPILED:generic_capc1005x50, F.Cu at (-144.8, 155.9)
- added C13: 100n, RPI_COMPILED:generic_capc1005x50, F.Cu at (-24.1, 128.2)
- added C130: 100n, RPI_COMPILED:generic_capc1005x50, F.Cu at (-144.8, 157.5)
- added C131: 100n, RPI_COMPILED:generic_capc1005x50, F.Cu at (-144.8, 159.0)
- added C132: 100n, RPI_COMPILED:generic_capc1005x50, F.Cu at (-144.8, 160.6)
- added C14: 100n, RPI_COMPILED:generic_capc1005x50, F.Cu at (-24.1, 129.8)
- added C15: 100n, RPI_COMPILED:generic_capc1005x50, F.Cu at (-24.1, 131.3)
- added C16: 100n, RPI_COMPILED:generic_capc1005x50, F.Cu at (-24.1, 132.9)
- added C17: 100n, RPI_COMPILED:generic_capc1005x50, F.Cu at (-21.6, 123.6)
- added C18: 100n, RPI_COMPILED:generic_capc1005x50, F.Cu at (-21.6, 125.1)
- added C19: 10u, RPI_COMPILED:generic_capc2012x125, F.Cu at (-21.4, 153.3)
- added C2: 100n, RPI_COMPILED:generic_capc1005x50, F.Cu at (-26.6, 123.6)
- added C20: 100n, RPI_COMPILED:generic_capc1005x50, F.Cu at (-21.6, 126.7)
- added C21: 100n, RPI_COMPILED:generic_capc1005x50, F.Cu at (-21.6, 128.2)
- added C23: 22uF, PixelBlit:C_0805, F.Cu at (-19.9, 84.2)
- added C24: 22uF, PixelBlit:C_0805, F.Cu at (-19.9, 87.3)
- added C25: 10uF, PixelBlit:C_0603, F.Cu at (-20.2, 70.3)
- added C26: 10uF, PixelBlit:C_0603, F.Cu at (-20.2, 72.6)
- added C27: 100nF, PixelBlit:C_0603, F.Cu at (-20.2, 74.8)
- added C28: 100nF, PixelBlit:C_0402, F.Cu at (-33.3, 117.0)
- added C29: 10uF, PixelBlit:C_0603, F.Cu at (-20.2, 77.1)
- added C3: 15p, RPI_COMPILED:generic_capc1005x50, F.Cu at (-26.6, 125.1)
- added C30: 100nF, PixelBlit:C_0603, F.Cu at (-20.2, 79.3)
- added C31: 10uF, PixelBlit:C_0603, F.Cu at (-20.2, 81.6)
- added C32: 10uF, PixelBlit:C_0805, F.Cu at (-19.9, 90.3)
- added C33: 47uF, PixelBlit:C_0805, F.Cu at (-19.9, 93.4)
- added C34: 100nF, PixelBlit:C_0402, F.Cu at (-77.4, 98.8)
- added C35: 100nF, PixelBlit:C_0402, F.Cu at (-77.4, 100.7)
- added C36: 100nF, PixelBlit:C_0402, F.Cu at (-77.4, 102.5)
- added C37: 100nF, PixelBlit:C_0402, F.Cu at (-77.4, 104.4)
- added C38: 100nF, PixelBlit:C_0402, F.Cu at (-77.4, 106.2)
- added C39: 100nF, PixelBlit:C_0402, F.Cu at (-77.4, 108.1)
- added C4: 15p, RPI_COMPILED:generic_capc1005x50, F.Cu at (-26.6, 126.7)
- added C40: 100nF, PixelBlit:C_0402, F.Cu at (-77.4, 109.9)
- added C41: 100nF, PixelBlit:C_0402, F.Cu at (-77.4, 111.8)
- added C6: 4.7u, RPI_COMPILED:generic_capc1005x50_wide, F.Cu at (-26.6, 128.2)
- added C7: 4.7u, RPI_COMPILED:generic_capc1005x50_wide, F.Cu at (-26.6, 129.8)
- added C8: 100n, RPI_COMPILED:generic_capc1005x50, F.Cu at (-26.6, 131.3)
- added C9: 4.7u, RPI_COMPILED:generic_capc1005x50, F.Cu at (-26.6, 132.9)
- added D1: B5819W, PixelBlit:D_SOD-123, F.Cu at (-20.4, 150.4)
- added D10: BZT52C15V, Diode_SMD:D_SOD-123, F.Cu at (-19.4, 108.5)
- added D11: SK6812MINI, LED_SMD:LED_SK6812MINI_PLCC4_3.5x3.5mm_P1.75mm, F.Cu at (-147.6, 147.4)
- added D12: SK6812MINI, LED_SMD:LED_SK6812MINI_PLCC4_3.5x3.5mm_P1.75mm, F.Cu at (-147.6, 152.6)
- added D13: SK6812MINI, LED_SMD:LED_SK6812MINI_PLCC4_3.5x3.5mm_P1.75mm, F.Cu at (-140.9, 137.2)
- added D14: SK6812MINI, LED_SMD:LED_SK6812MINI_PLCC4_3.5x3.5mm_P1.75mm, F.Cu at (-140.9, 142.3)
- added D15: SK6812MINI, LED_SMD:LED_SK6812MINI_PLCC4_3.5x3.5mm_P1.75mm, F.Cu at (-140.9, 147.4)
- added D16: SK6812MINI, LED_SMD:LED_SK6812MINI_PLCC4_3.5x3.5mm_P1.75mm, F.Cu at (-140.9, 152.6)
- added D17: SK6812MINI, LED_SMD:LED_SK6812MINI_PLCC4_3.5x3.5mm_P1.75mm, F.Cu at (-134.2, 137.2)
- added D18: SK6812MINI, LED_SMD:LED_SK6812MINI_PLCC4_3.5x3.5mm_P1.75mm, F.Cu at (-134.2, 142.3)
- added D19: SK6812MINI, LED_SMD:LED_SK6812MINI_PLCC4_3.5x3.5mm_P1.75mm, F.Cu at (-134.2, 147.4)
- added D2: USBLC6-2SC6, PixelBlit:SOT-23-6_L2.9-W1.6-P0.95-LS2.8-BL, F.Cu at (-25.4, 152.1)
- added D20: SK6812MINI, LED_SMD:LED_SK6812MINI_PLCC4_3.5x3.5mm_P1.75mm, F.Cu at (-134.2, 152.6)
- added D21: SK6812MINI, LED_SMD:LED_SK6812MINI_PLCC4_3.5x3.5mm_P1.75mm, F.Cu at (-127.5, 137.2)
- added D22: SK6812MINI, LED_SMD:LED_SK6812MINI_PLCC4_3.5x3.5mm_P1.75mm, F.Cu at (-127.5, 142.3)
- added D23: SK6812MINI, LED_SMD:LED_SK6812MINI_PLCC4_3.5x3.5mm_P1.75mm, F.Cu at (-127.5, 147.4)
- added D24: SK6812MINI, LED_SMD:LED_SK6812MINI_PLCC4_3.5x3.5mm_P1.75mm, F.Cu at (-127.5, 152.6)
- added D3: SK6812MINI, LED_SMD:LED_SK6812MINI_PLCC4_3.5x3.5mm_P1.75mm, F.Cu at (-147.6, 137.2)
- added D4: B5819W, PixelBlit:D_SOD-123, F.Cu at (-25.2, 108.5)
- added D5: SS34, PCM_JLCPCB:D_SMA, F.Cu at (-18.0, 53.3)
- added D6: SS34, PCM_JLCPCB:D_SMA, F.Cu at (-18.0, 57.8)
- added D7: SS34, PCM_JLCPCB:D_SMA, F.Cu at (-18.0, 62.4)
- added D8: SS34, PCM_JLCPCB:D_SMA, F.Cu at (-18.0, 66.9)
- added D9: SK6812MINI, LED_SMD:LED_SK6812MINI_PLCC4_3.5x3.5mm_P1.75mm, F.Cu at (-147.6, 142.3)
- added F1: 3557-2, EasyEDA:FUSE-TH_4P-L19.8-W6.7_3557-2, F.Cu at (232.9, 57.5)
- added F10: 1812L400/16GR, EasyEDA:F1812, F.Cu at (193.1, 34.9)
- added F11: 1812L400/16GR, EasyEDA:F1812, F.Cu at (171.8, 34.9)
- added F12: 1812L400/16GR, EasyEDA:F1812, F.Cu at (150.4, 34.9)
- added F13: 1812L400/16GR, EasyEDA:F1812, F.Cu at (129.1, 34.9)
- added F14: 1812L400/16GR, EasyEDA:F1812, F.Cu at (107.7, 34.9)
- added F15: 1812L400/16GR, EasyEDA:F1812, F.Cu at (86.4, 34.9)
- added F16: 1812L400/16GR, EasyEDA:F1812, F.Cu at (215.0, 45.5)
- added F17: 1812L400/16GR, EasyEDA:F1812, F.Cu at (-87.4, 53.6)
- added F18: 1812L400/16GR, EasyEDA:F1812, F.Cu at (-87.4, 58.8)
- added F19: 1812L400/16GR, EasyEDA:F1812, F.Cu at (-87.4, 64.0)
- added F2: 3557-2, EasyEDA:FUSE-TH_4P-L19.8-W6.7_3557-2, F.Cu at (232.7, 81.0)
- added F20: 1812L400/16GR, EasyEDA:F1812, F.Cu at (-87.4, 69.2)
- added F21: 1812L400/16GR, EasyEDA:F1812, F.Cu at (-87.4, 74.4)
- added F22: 1812L400/16GR, EasyEDA:F1812, F.Cu at (-87.4, 79.7)
- added F23: 1812L400/16GR, EasyEDA:F1812, F.Cu at (-87.4, 84.9)
- added F24: 1812L400/16GR, EasyEDA:F1812, F.Cu at (-87.4, 90.1)
- added F25: 1812L400/16GR, EasyEDA:F1812, F.Cu at (-87.4, 95.3)
- added F26: 1812L400/16GR, EasyEDA:F1812, F.Cu at (-79.2, 53.6)
- added F27: 1812L400/16GR, EasyEDA:F1812, F.Cu at (-79.2, 58.8)
- added F28: 1812L400/16GR, EasyEDA:F1812, F.Cu at (-79.2, 64.0)
- added F29: 1812L400/16GR, EasyEDA:F1812, F.Cu at (-79.2, 69.2)
- added F3: 3557-2, EasyEDA:FUSE-TH_4P-L19.8-W6.7_3557-2, F.Cu at (233.0, 104.5)
- added F30: 1812L400/16GR, EasyEDA:F1812, F.Cu at (-79.2, 74.4)
- added F31: 1812L400/16GR, EasyEDA:F1812, F.Cu at (-79.2, 79.7)
- added F32: 1812L400/16GR, EasyEDA:F1812, F.Cu at (-79.2, 84.9)
- added F33: 1812L400/16GR, EasyEDA:F1812, F.Cu at (-79.2, 90.1)
- added F34: 1812L400/16GR, EasyEDA:F1812, F.Cu at (-79.2, 95.3)
- added F35: 1812L400/16GR, EasyEDA:F1812, F.Cu at (-71.0, 53.6)
- added F36: 1812L400/16GR, EasyEDA:F1812, F.Cu at (-71.0, 58.8)
- added F37: 1812L400/16GR, EasyEDA:F1812, F.Cu at (-71.0, 64.0)
- added F38: 1812L400/16GR, EasyEDA:F1812, F.Cu at (-71.0, 69.2)
- added F39: 1812L400/16GR, EasyEDA:F1812, F.Cu at (-71.0, 74.4)
- added F4: 3557-2, EasyEDA:FUSE-TH_4P-L19.8-W6.7_3557-2, F.Cu at (233.2, 128.2)
- added F5: 3557-2, EasyEDA:FUSE-TH_4P-L19.8-W6.7_3557-2, F.Cu at (224.2, 59.0)
- added F6: 3557-2, EasyEDA:FUSE-TH_4P-L19.8-W6.7_3557-2, F.Cu at (224.0, 93.5)
- added F7: 3557-2, EasyEDA:FUSE-TH_4P-L19.8-W6.7_3557-2, F.Cu at (224.0, 126.2)
- added F8: 1812L400/16GR, EasyEDA:F1812, F.Cu at (237.5, 35.0)
- added F9: 1812L400/16GR, EasyEDA:F1812, F.Cu at (214.5, 34.9)
- added H1: MountingHole_Pad, PixelBlit:MountingHole_3.2mm_M3_Pad_Via, F.Cu at (62.7, 34.7)
- added H2: MountingHole_Pad, PixelBlit:MountingHole_3.2mm_M3_Pad_Via, F.Cu at (62.7, 150.5)
- added H3: MountingHole_Pad, PixelBlit:MountingHole_3.2mm_M3_Pad_Via, F.Cu at (253.4, 35.5)
- added H4: MountingHole_Pad, PixelBlit:MountingHole_3.2mm_M3_Pad_Via, F.Cu at (252.8, 150.5)
- added J1: Conn_01x03_Pin, Connector_PinHeader_2.54mm:PinHeader_1x03_P2.54mm_Vertical, F.Cu at (-25.6, 142.6)
- added J10: DB301V-3.5-3P-GN, PixelBlit:CONN-TH_DB301V-3.5-3P-GN, F.Cu at (160.9, 39.0)
- added J11: DB301V-3.5-3P-GN, PixelBlit:CONN-TH_DB301V-3.5-3P-GN, F.Cu at (139.6, 39.0)
- added J12: DB301V-3.5-3P-GN, PixelBlit:CONN-TH_DB301V-3.5-3P-GN, F.Cu at (118.2, 39.0)
- added J13: DB301V-3.5-3P-GN, PixelBlit:CONN-TH_DB301V-3.5-3P-GN, F.Cu at (96.9, 39.0)
- added J14: DB301V-3.5-3P-GN, PixelBlit:CONN-TH_DB301V-3.5-3P-GN, F.Cu at (75.5, 39.0)
- added J15: DB301V-3.5-3P-GN, PixelBlit:CONN-TH_DB301V-3.5-3P-GN, F.Cu at (214.0, 54.0)
- added J16: DB301V-3.5-3P-GN, PixelBlit:CONN-TH_DB301V-3.5-3P-GN, F.Cu at (193.5, 54.0)
- added J17: DB301V-3.5-3P-GN, PixelBlit:CONN-TH_DB301V-3.5-3P-GN, F.Cu at (172.5, 54.0)
- added J18: DB301V-3.5-3P-GN, PixelBlit:CONN-TH_DB301V-3.5-3P-GN, F.Cu at (151.0, 54.0)
- added J19: DB301V-3.5-3P-GN, PixelBlit:CONN-TH_DB301V-3.5-3P-GN, F.Cu at (129.5, 54.0)
- added J2: Conn_01x02_Pin, Connector_PinHeader_2.54mm:PinHeader_1x02_P2.54mm_Vertical, F.Cu at (-20.1, 157.1)
- added J20: DB301V-3.5-3P-GN, PixelBlit:CONN-TH_DB301V-3.5-3P-GN, F.Cu at (108.0, 54.0)
- added J21: DB301V-3.5-3P-GN, PixelBlit:CONN-TH_DB301V-3.5-3P-GN, F.Cu at (86.5, 54.0)
- added J22: DB301V-3.5-3P-GN, PixelBlit:CONN-TH_DB301V-3.5-3P-GN, F.Cu at (66.0, 54.0)
- added J23: DB301V-3.5-3P-GN, PixelBlit:CONN-TH_DB301V-3.5-3P-GN, F.Cu at (-131.7, 109.7)
- added J24: DB301V-3.5-3P-GN, PixelBlit:CONN-TH_DB301V-3.5-3P-GN, F.Cu at (-131.7, 117.5)
- added J25: DB301V-3.5-3P-GN, PixelBlit:CONN-TH_DB301V-3.5-3P-GN, F.Cu at (-118.9, 55.0)
- added J26: DB301V-3.5-3P-GN, PixelBlit:CONN-TH_DB301V-3.5-3P-GN, F.Cu at (-118.9, 62.8)
- added J27: DB301V-3.5-3P-GN, PixelBlit:CONN-TH_DB301V-3.5-3P-GN, F.Cu at (-118.9, 70.7)
- added J28: DB301V-3.5-3P-GN, PixelBlit:CONN-TH_DB301V-3.5-3P-GN, F.Cu at (-118.9, 78.5)
- added J29: DB301V-3.5-3P-GN, PixelBlit:CONN-TH_DB301V-3.5-3P-GN, F.Cu at (-118.9, 86.3)
- added J3: DBT50G-9.5-2P, EasyEDA:CONN-TH_2P-P9.50_DBT50G-9.5-2P, F.Cu at (242.2, 57.5)
- added J30: DB301V-3.5-3P-GN, PixelBlit:CONN-TH_DB301V-3.5-3P-GN, F.Cu at (-118.9, 94.1)
- added J31: DB301V-3.5-3P-GN, PixelBlit:CONN-TH_DB301V-3.5-3P-GN, F.Cu at (-118.9, 101.9)
- added J32: DB301V-3.5-3P-GN, PixelBlit:CONN-TH_DB301V-3.5-3P-GN, F.Cu at (-118.9, 109.7)
- added J33: DB301V-3.5-3P-GN, PixelBlit:CONN-TH_DB301V-3.5-3P-GN, F.Cu at (-118.9, 117.5)
- added J34: DB301V-3.5-3P-GN, PixelBlit:CONN-TH_DB301V-3.5-3P-GN, F.Cu at (-106.1, 55.0)
- added J35: DB301V-3.5-3P-GN, PixelBlit:CONN-TH_DB301V-3.5-3P-GN, F.Cu at (-106.1, 62.8)
- added J36: DB301V-3.5-3P-GN, PixelBlit:CONN-TH_DB301V-3.5-3P-GN, F.Cu at (-106.1, 70.7)
- added J37: DB301V-3.5-3P-GN, PixelBlit:CONN-TH_DB301V-3.5-3P-GN, F.Cu at (-106.1, 78.5)
- added J38: 2.54-1*4, PixelBlit:HDR-TH_4P-P2.54-V-M-1, F.Cu at (-37.5, 108.7)
- added J39: DB301V-3.5-3P-GN, PixelBlit:CONN-TH_DB301V-3.5-3P-GN, F.Cu at (-106.1, 86.3)
- added J4: DBT50G-9.5-2P, EasyEDA:CONN-TH_2P-P9.50_DBT50G-9.5-2P, F.Cu at (242.2, 81.0)
- added J5: DBT50G-9.5-2P, EasyEDA:CONN-TH_2P-P9.50_DBT50G-9.5-2P, F.Cu at (242.2, 104.5)
- added J6: DBT50G-9.5-2P, EasyEDA:CONN-TH_2P-P9.50_DBT50G-9.5-2P, F.Cu at (242.2, 128.0)
- added J7: DB301V-3.5-3P-GN, PixelBlit:CONN-TH_DB301V-3.5-3P-GN, F.Cu at (225.0, 39.0)
- added J8: DB301V-3.5-3P-GN, PixelBlit:CONN-TH_DB301V-3.5-3P-GN, F.Cu at (203.6, 39.0)
- added J9: DB301V-3.5-3P-GN, PixelBlit:CONN-TH_DB301V-3.5-3P-GN, F.Cu at (182.3, 39.0)
- added JP1: SolderJumper_2_Bridged, Jumper:SolderJumper-2_P1.3mm_Bridged_RoundedPad1.0x1.5mm, F.Cu at (-36.9, 117.9)
- added L1: 3.3u, RPI_COMPILED:abracon_aota-b201610s3r3-101-t, F.Cu at (-20.4, 167.3)
- added L2: FXL0420-1R5-M, EasyEDA:IND-SMD_L4.4-W4.2, F.Cu at (-35.5, 113.4)
- added PWR_LED1: Red, PixelBlit:D_0603, F.Cu at (-41.1, 111.9)
- added PWR_LED2: Red, PixelBlit:D_0603, F.Cu at (-41.1, 114.5)
- added PWR_LED3: Red, PixelBlit:D_0603, F.Cu at (-41.1, 117.1)
- added R1: 10k, RPI_COMPILED:generic_resc1005x35, F.Cu at (-21.6, 129.8)
- added R10: 0, RPI_COMPILED:generic_resc1005x35, F.Cu at (-19.1, 131.3)
- added R11: 5.1kΩ, PixelBlit:R_0402, F.Cu at (-52.7, 161.1)
- added R12: 5.1kΩ, PixelBlit:R_0402, F.Cu at (-52.7, 163.0)
- added R13: 10kΩ, PixelBlit:R_0603, F.Cu at (-30.0, 108.0)
- added R14: 560kΩ, PixelBlit:R_0402, F.Cu at (-26.8, 111.1)
- added R15: 100kΩ, PixelBlit:R_0402, F.Cu at (-26.8, 113.0)
- added R16: 100kΩ, PixelBlit:R_0603, F.Cu at (-30.0, 110.2)
- added R17: 100kΩ, PixelBlit:R_0603, F.Cu at (-30.0, 112.5)
- added R18: 1kΩ, PixelBlit:R_0402, F.Cu at (-26.8, 114.8)
- added R19: 47Ω, PixelBlit:R_0402, F.Cu at (-142.1, 160.7)
- added R2: 1k, RPI_COMPILED:generic_resc1005x35, F.Cu at (-21.6, 131.3)
- added R20: 2.2kΩ, Resistor_SMD:R_0603_1608Metric, F.Cu at (-23.3, 114.0)
- added R21: 47Ω, PixelBlit:R_0402, F.Cu at (-88.8, 98.8)
- added R24: 47Ω, PixelBlit:R_0402, F.Cu at (-88.8, 100.7)
- added R25: 47Ω, PixelBlit:R_0402, F.Cu at (-88.8, 102.5)
- added R26: 47Ω, PixelBlit:R_0402, F.Cu at (-88.8, 104.4)
- added R27: 47Ω, PixelBlit:R_0402, F.Cu at (-88.8, 106.2)
- added R28: 47Ω, PixelBlit:R_0402, F.Cu at (-88.8, 108.1)
- added R29: 47Ω, PixelBlit:R_0402, F.Cu at (-88.8, 109.9)
- added R3: 33, RPI_COMPILED:generic_resc1005x35, F.Cu at (-21.6, 132.9)
- added R30: 47Ω, PixelBlit:R_0402, F.Cu at (-88.8, 111.8)
- added R31: 47Ω, PixelBlit:R_0402, F.Cu at (-88.8, 113.6)
- added R32: 47Ω, PixelBlit:R_0402, F.Cu at (-85.9, 98.8)
- added R33: 47Ω, PixelBlit:R_0402, F.Cu at (-85.9, 100.7)
- added R34: 47Ω, PixelBlit:R_0402, F.Cu at (-85.9, 102.5)
- added R35: 47Ω, PixelBlit:R_0402, F.Cu at (-85.9, 104.4)
- added R36: 47Ω, PixelBlit:R_0402, F.Cu at (-85.9, 106.2)
- added R37: 47Ω, PixelBlit:R_0402, F.Cu at (-85.9, 108.1)
- added R38: 47Ω, PixelBlit:R_0402, F.Cu at (-85.9, 109.9)
- added R39: 47Ω, PixelBlit:R_0402, F.Cu at (-85.9, 111.8)
- added R4: 1k, RPI_COMPILED:generic_resc1005x35, F.Cu at (-19.1, 123.6)
- added R40: 47Ω, PixelBlit:R_0402, F.Cu at (-85.9, 113.6)
- added R41: 47Ω, PixelBlit:R_0402, F.Cu at (-83.1, 98.8)
- added R42: 47Ω, PixelBlit:R_0402, F.Cu at (-83.1, 100.7)
- added R43: 47Ω, PixelBlit:R_0402, F.Cu at (-83.1, 102.5)
- added R44: 47Ω, PixelBlit:R_0402, F.Cu at (-83.1, 104.4)
- added R45: 47Ω, PixelBlit:R_0402, F.Cu at (-83.1, 106.2)
- added R46: 47Ω, PixelBlit:R_0402, F.Cu at (-83.1, 108.1)
- added R47: 47Ω, PixelBlit:R_0402, F.Cu at (-83.1, 109.9)
- added R48: 47Ω, PixelBlit:R_0402, F.Cu at (-83.1, 111.8)
- added R49: 47Ω, PixelBlit:R_0402, F.Cu at (-83.1, 113.6)
- added R5: 8.2kΩ, Resistor_SMD:R_0603_1608Metric, F.Cu at (-23.3, 111.5)
- added R50: 47Ω, PixelBlit:R_0402, F.Cu at (-80.2, 98.8)
- added R51: 47Ω, PixelBlit:R_0402, F.Cu at (-80.2, 100.7)
- added R52: 47Ω, PixelBlit:R_0402, F.Cu at (-80.2, 102.5)
- added R53: 47Ω, PixelBlit:R_0402, F.Cu at (-80.2, 104.4)
- added R54: 47Ω, PixelBlit:R_0402, F.Cu at (-80.2, 106.2)
- added R6: 1k, RPI_COMPILED:generic_resc1005x35, F.Cu at (-19.1, 125.1)
- added R7: 27, RPI_COMPILED:generic_resc1005x35, F.Cu at (-19.1, 126.7)
- added R8: 27, RPI_COMPILED:generic_resc1005x35, F.Cu at (-19.1, 128.2)
- added R9: 0, RPI_COMPILED:generic_resc1005x35, F.Cu at (-19.1, 129.8)
- added R94: 10kΩ, PixelBlit:R_0603, F.Cu at (-24.2, 156.0)
- added R95: 10kΩ, PixelBlit:R_0603, F.Cu at (-24.2, 158.2)
- added R96: 10kΩ, PixelBlit:R_0603, F.Cu at (-24.2, 160.5)
- added R97: 10kΩ, PixelBlit:R_0603, F.Cu at (-24.2, 162.7)
- added R98: 470Ω, PixelBlit:R_0603, F.Cu at (-24.2, 165.0)
- added SW1: 434133025816, RPI_COMPILED:wurthelek_434133025816, F.Cu at (-20.4, 142.4)
- added SW2: 434133025816, RPI_COMPILED:wurthelek_434133025816, F.Cu at (-20.4, 146.6)
- added TP2: TestPoint, PixelBlit:TestPoint_Pad_1.0x1.0mm, F.Cu at (-30.3, 115.1)
- added TP3: TestPoint, PixelBlit:TestPoint_Pad_1.0x1.0mm, F.Cu at (-30.3, 118.2)
- added U1: RP2350B, RPI_COMPILED:rpi_rp2350b_vias, F.Cu at (-31.9, 160.8)
- added U10: SN74LVC8T245PWR, PixelBlit:TSSOP-24_L7.8-W4.4-P0.65-LS6.4-BL, F.Cu at (-94.8, 119.6)
- added U11: SN74LVC8T245PWR, PixelBlit:TSSOP-24_L7.8-W4.4-P0.65-LS6.4-BL, F.Cu at (-94.8, 128.3)
- added U2: RPI RM2, RF_Module:RMC20452T, F.Cu at (66.5, 117.8)
- added U3: W25Q128JVSIQ, RPI_COMPILED:generic_soic127p790x195-8, F.Cu at (-22.9, 137.2)
- added U4: SN74LVC1T45DBV, Package_TO_SOT_SMD:SOT-23-6, F.Cu at (-140.9, 157.5)
- added U5: TPS63070RNMR, PixelBlit:VQFN-HR-15_L3.0-W2.5-P0.50-BL_TPS63070RNMR, F.Cu at (-19.0, 116.7)
- added U6: ~, PixelBlit:SOT-23-5_L3.0-W1.7-P0.95-LS2.8-BR, F.Cu at (-19.0, 112.3)
- added U7: SN74LVC8T245PWR, PixelBlit:TSSOP-24_L7.8-W4.4-P0.65-LS6.4-BL, F.Cu at (-94.8, 102.2)
- added U8: SN74LVC8T245PWR, PixelBlit:TSSOP-24_L7.8-W4.4-P0.65-LS6.4-BL, F.Cu at (-94.8, 110.9)
- added U9: DS3231SN, Package_SO:SOIC-16W_7.5x10.3mm_P1.27mm, F.Cu at (-44.3, 160.9)
- added USB1: TYPE-C 16PIN 2MD(073), PixelBlit:USB-C-SMD_TYPE-C-6PIN-2MD-073, F.Cu at (-59.5, 163.6)
- added X1: 12MHz, RPI_COMPILED:generic_xtalcc320x250x80-4, F.Cu at (-19.6, 163.9)
Other:
- board size 181 x 125 mm -> 200 x 125 mm
