File: Power.kicad_sch (KiCad schematic)
At the start: 46 parts, among them J3 DBT50G-9.5-2P, J38 2.54-1*4, J4 DBT50G-9.5-2P, J5 DBT50G-9.5-2P, J6 DBT50G-9.5-2P, U5 TPS63070RNMR

Commit message: Start PCB layout and add mounting holes
Footprints placed on the board, H1-H4 mounting holes added to the
schematic, and schematic updates to Output and Power sheets.

Co-Authored-By: Claude Opus 5.5 <noreply@anthropic.com>
Parts:
- JP1: footprint (none) -> Jumper:SolderJumper-2_P1.3mm_Bridged_RoundedPad1.0x1.5mm
Changed lines of the file:
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@@
 			)
 		)
-		(property "Footprint" ""
+		(property "Footprint" "Jumper:SolderJumper-2_P1.3mm_Bridged_RoundedPad1.0x1.5mm"
 			(at 110.49 153.67 0)
 			(hide yes)
