File: universal-strip-controller.kicad_sch (KiCad schematic)
At the start: 50 parts, among them J1 Conn_01x03_Pin, J2 Conn_01x02_Pin, SW1 434133025816, SW2 434133025816, U1 RP2350B, U2 RPI RM2, U3 W25Q128JVSIQ, U9 DS3231SN, X1 12MHz

Commit message: Start PCB layout and add mounting holes
Footprints placed on the board, H1-H4 mounting holes added to the
schematic, and schematic updates to Output and Power sheets.

Co-Authored-By: Claude Opus 5.5 <noreply@anthropic.com>
Parts:
- added H1, H2, H3, H4: MountingHole_Pad, PixelBlit:MountingHole_3.2mm_M3_Pad_Via, symbol PixelBlit:MountingHole_Pad
Connections:
- net GND: now also H1.1, H2.1, H3.1, H4.1
